File: Eagle/FmBoard/SI4689_Fm_Module.sch (EAGLE design)
At the start: 69 parts, among them IC1 TPS79318DBVR, IC2 SI4688-A10-GM, U1 TXS0104EPWR, U2 3.3V/150mA, X2 19.2MHz

Commit message: Updated to the now working v1.7 of the radio module Made Radio Module arudino compatible so that it can be plugged directly into the arudino Moved to a S25FL132K0XMFI041 flash chip due to being cheaper and easier to program.
Parts:
- removed D1: ESD9L5.0, generisch:ESD9L5.0
- removed ISP: AVRISP-6, adafruit:AVRISP-6
- removed SJ1: SOLDERJUMPERNC, SparkFun-Retired:SOLDERJUMPERNC
- removed SMODE: (no value), SparkFun-Retired:SOLDERJUMPER_2WAYS
- added D3: (no value), adafruit:DIODESOD-323F
- added D4: (no value), SparkFun-DiscreteSemi:DIODESOD523
- added ISP1: AVRISP-6, adafruit:AVRISP-6
- added U$1: SWITCH_SPDTMOUSER, SparkFun-Electromechanical:SWITCH_SPDTMOUSER
- FLASH: value SST25VF016BSOIC -> SPI_FLASH-X25XXSMD; device john:SST25VF016BSOIC -> SparkFun-DigitalIC:SPI_FLASH-X25XXSMD
- IC2: value SI4688-A10-GM -> SI4689GM; device SI4688-A10-GM:SI4688-A10-GM -> john:SI4689GM
Connections:
- removed net SPI0_CE0_N: CONTROL.1, R5.1, U1.B4
- new net N$10: CHIP.1, D3.C
- new net N$19: D2.A, POWER.1
- new net SPI0_SSB: CONTROL.3, R5.1, U1.B4
- net +1V8: now also U$1.S; no longer SMODE.3
- net 3.3V: now also D4.A; no longer D2.A, SJ1.2
- net FLASH_CE: now also FLASH.CS, ISP1.RST; no longer FLASH.CE#, ISP.RST
- net FLASH_SCK: now also ISP1.SCK; no longer ISP.SCK
- net FLASH_SI: now also FLASH.MOSI, ISP1.MOSI; no longer FLASH.SI, ISP.MOSI
- net FLASH_SO: now also FLASH.MISO, ISP1.MISO; no longer FLASH.SO, ISP.MISO
- net FLASH_VIN: now also D4.C, FLASH.VCC, ISP1.VCC; no longer D2.C, FLASH.VDD, ISP.VCC
- net GND: now also FLASH.GND, ISP1.GND, U$1.O; no longer D1.A, FLASH.VSS, ISP.GND, SMODE.1
- net INT: now also D3.A; no longer CHIP.1
- net LDO_IN: now also D2.C; no longer POWER.1, SJ1.1
- net N$14: now also FLASH.WP; no longer FLASH.WP#
- net N$17: now also U$1.P; no longer SMODE.2
- net RF_IN: no longer D1.C
- net SPI0_MOSI: now also CONTROL.2; no longer CONTROL.3
- net SPI0_SCLK: now also CONTROL.1; no longer CONTROL.2
Other:
- moved on the sheet: D2, FLASH
